File: pcb/AAfilter.sch (KiCad schematic (older format))
At the start: 10 parts

Commit message: clean up, label sub circuit blocks in silkscreen document the expected clock and baseband amplitudes based on opamp gains
Changed lines of the file:
@@
 $Descr A4 11693 8268
 encoding utf-8
-Sheet 6 6
+Sheet 5 6
 Title ""
 Date ""
@@
 AR Path="/5FB3742F/5FBD65F9/5FBFCF8A" Ref="C?"  Part="1"
 AR Path="/5FB3742F/5FBDAA40/5FBFCF8A" Ref="C88"  Part="1"
-F 0 "C88" H 3765 3196 50  0000 L CNN
+F 0 "C76" H 3765 3196 50  0000 L CNN
 F 1 "85p" H 3765 3105 50  0000 L CNN
 F 2 "Capacitor_SMD:C_0603_1608Metric" H 3688 3000 50  0001 C CNN
@@
 AR Path="/5FB3742F/5FBD65F9/5FBFCF84" Ref="L?"  Part="1"
 AR Path="/5FB3742F/5FBDAA40/5FBFCF84" Ref="L30"  Part="1"
-F 0 "L30" V 2340 3300 50  0000 C CNN
+F 0 "L12" V 2340 3300 50  0000 C CNN
 F 1 "732n" V 2249 3300 50  0000 C CNN
 F 2 "Inductor_SMD:L_0603_1608Metric" H 2150 3300 50  0001 C CNN
@@
 AR Path="/5FB3742F/5FBD65F9/5FBFD013" Ref="C?"  Part="1"
 AR Path="/5FB3742F/5FBDAA40/5FBFD013" Ref="C80"  Part="1"
-F 0 "C80" H 1965 3196 50  0000 L CNN
+F 0 "C68" H 1965 3196 50  0000 L CNN
 F 1 "85p" H 1965 3105 50  0000 L CNN
 F 2 "Capacitor_SMD:C_0603_1608Metric" H 1888 3000 50  0001 C CNN
@@
 AR Path="/5FB3742F/5FBD65F9/5FBFD014" Ref="L?"  Part="1"
 AR Path="/5FB3742F/5FBDAA40/5FBFD014" Ref="L28"  Part="1"
-F 0 "L28" V 2340 3000 50  0000 C CNN
+F 0 "L10" V 2340 3000 50  0000 C CNN
 F 1 "732n" V 2249 3000 50  0000 C CNN
 F 2 "Inductor_SMD:L_0603_1608Metric" H 2150 3000 50  0001 C CNN
@@
 AR Path="/5FB3742F/5FBD65F9/5FBA6C76" Ref="C?"  Part="1"
 AR Path="/5FB3742F/5FBDAA40/5FBA6C76" Ref="C84"  Part="1"
-F 0 "C84" H 3165 3196 50  0000 L CNN
+F 0 "C72" H 3165 3196 50  0000 L CNN
 F 1 "187p" H 3165 3105 50  0000 L CNN
 F 2 "Capacitor_SMD:C_0603_1608Metric" H 3088 3000 50  0001 C CNN
@@
 AR Path="/5FB3742F/5FBD65F9/5FBA6C88" Ref="L?"  Part="1"
 AR Path="/5FB3742F/5FBDAA40/5FBA6C88" Ref="L38"  Part="1"
-F 0 "L38" V 3540 3000 50  0000 C CNN
+F 0 "L20" V 3540 3000 50  0000 C CNN
 F 1 "732n" V 3449 3000 50  0000 C CNN
 F 2 "Inductor_SMD:L_0603_1608Metric" H 3350 3000 50  0001 C CNN
@@
 AR Path="/5FB3742F/5FBD65F9/5FBA6C70" Ref="L?"  Part="1"
 AR Path="/5FB3742F/5FBDAA40/5FBA6C70" Ref="L35"  Part="1"
-F 0 "L35" V 2940 3300 50  0000 C CNN
+F 0 "L17" V 2940 3300 50  0000 C CNN
 F 1 "866n" V 2849 3300 50  0000 C CNN
 F 2 "Inductor_SMD:L_0603_1608Metric" H 2750 3300 50  0001 C CNN
@@
 AR Path="/5FB3742F/5FBD65F9/5FBFD016" Ref="C?"  Part="1"
 AR Path="/5FB3742F/5FBDAA40/5FBFD016" Ref="C83"  Part="1"
-F 0 "C83" H 2565 3196 50  0000 L CNN
+F 0 "C71" H 2565 3196 50  0000 L CNN
 F 1 "187p" H 2565 3105 50  0000 L CNN
 F 2 "Capacitor_SMD:C_0603_1608Metric" H 2488 3000 50  0001 C CNN
@@
 AR Path="/5FB3742F/5FBD65F9/5FBA6C6A" Ref="L?"  Part="1"
 AR Path="/5FB3742F/5FBDAA40/5FBA6C6A" Ref="L32"  Part="1"
-F 0 "L32" V 2940 3000 50  0000 C CNN
+F 0 "L14" V 2940 3000 50  0000 C CNN
 F 1 "866n" V 2849 3000 50  0000 C CNN
 F 2 "Inductor_SMD:L_0603_1608Metric" H 2750 3000 50  0001 C CNN
@@
 AR Path="/5FB3742F/5FBD65F9/5FBA6C7C" Ref="L?"  Part="1"
 AR Path="/5FB3742F/5FBDAA40/5FBA6C7C" Ref="L41"  Part="1"
-F 0 "L41" V 3540 3300 50  0000 C CNN
+F 0 "L23" V 3540 3300 50  0000 C CNN
 F 1 "732n" V 3449 3300 50  0000 C CNN
 F 2 "Inductor_SMD:L_0603_1608Metric" H 3350 3300 50  0001 C CNN

Commit message: populate LCSC BOM for JLCPCB assembly
Parts:
- C68, C76: value 85p -> 330p; LCSC (none) -> C1664
- C71, C72: value 187p -> 680p; LCSC (none) -> C30816
- L10, L12, L20, L23: value 732n -> 330n; LCSC (none) -> C46859
- L14, L17: value 866n -> 470n; LCSC (none) -> C21307
