File: pcb/iq_siggen.sch (KiCad schematic (older format))
At the start: 94 parts, among them J1 J3 - BANK0, J10 Barrel_Jack, J11 Conn_Coaxial, J12 Conn_01x01_Male, J13 Conn_01x01_Male, J14 Conn_01x01_Male, J15 Conn_01x01_Male, J16 Conn_01x01_Male, J17 Conn_01x01_Male, J2 J4 - BANK1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

Commit message: fill out more components in BOM with LCSC parts
Parts:
- C6: footprint Capacitor_Tantalum_SMD:CP_EIA-7343-20_Kemet-V_Pad2.25x2.55mm_HandSolder -> Capacitor_Tantalum_SMD:CP_EIA-7343-43_Kemet-X_Pad2.25x2.55mm_HandSolder; LCSC (none) -> C7231
Changed lines of the file:
@@
 F 0 "C6" H 10518 1046 50  0000 L CNN
 F 1 "220u" H 10518 955 50  0000 L CNN
-F 2 "Capacitor_Tantalum_SMD:CP_EIA-7343-20_Kemet-V_Pad2.25x2.55mm_HandSolder" H 10438 850 50  0001 C CNN
+F 2 "Capacitor_Tantalum_SMD:CP_EIA-7343-43_Kemet-X_Pad2.25x2.55mm_HandSolder" H 10438 850 50  0001 C CNN
 F 3 "~" H 10400 1000 50  0001 C CNN
+F 4 "C7231" H 10400 1000 50  0001 C CNN "LCSC"
 	1    10400 1000
 	1    0    0    -1
