File: pcb/sigma_delta_adc_board/sigma_delta_adc_board.sch (KiCad schematic (older format))
At the start: 28 parts, among them J1 AudioJack3_Ground_SwitchTR, J2 Conn_01x02, J3 Conn_01x02, U1 MCP6002-xP, U2 FPGA LVDS INPUT

Commit message: finish the board
Parts:
- removed C9: 10u, symbol Device:CP
- removed U2: FPGA LVDS INPUT, symbol Amplifier_Operational:MCP6002-xP
- added J4: Conn_02x05_Counter_Clockwise, Connector_PinSocket_2.54mm:PinSocket_2x05_P2.54mm_Vertical, symbol Connector_Generic:Conn_02x05_Odd_Even
- added TP8, TP9: TestPoint, TestPoint:TestPoint_Pad_D1.0mm, symbol Connector:TestPoint
- added unit 3 of U1
- added unit 2 of U1
- C1, C5: footprint (none) -> Capacitor_THT:C_Disc_D5.0mm_W2.5mm_P5.00mm
- C2, C4: value C -> 1u; footprint (none) -> Capacitor_SMD:C_0805_2012Metric_Pad1.18x1.45mm_HandSolder
- C3: value C -> 10u; footprint (none) -> Capacitor_THT:C_Disc_D5.0mm_W2.5mm_P5.00mm
- C6, C7: value C -> 0.1u; footprint (none) -> Capacitor_SMD:C_0805_2012Metric_Pad1.18x1.45mm_HandSolder
- C8: footprint (none) -> Capacitor_SMD:C_0805_2012Metric_Pad1.18x1.45mm_HandSolder
- J1: footprint (none) -> sigma_delta_adc_board:STX-3120-5B
- J2, J3: footprint (none) -> Connector_PinHeader_2.54mm:PinHeader_1x02_P2.54mm_Vertical
- JP1: footprint (none) -> Jumper:SolderJumper-3_P1.3mm_Open_RoundedPad1.0x1.5mm_NumberLabels
- R1, R2, R3, R4: footprint (none) -> Resistor_SMD:R_0805_2012Metric_Pad1.20x1.40mm_HandSolder
- R5, R6: value 1k -> R; footprint (none) -> Resistor_SMD:R_0805_2012Metric_Pad1.20x1.40mm_HandSolder
- TP1, TP2, TP3, TP4, TP5, TP6, TP7: footprint (none) -> Connector_PinHeader_2.54mm:PinHeader_1x01_P2.54mm_Vertical
- U1: footprint (none) -> Package_DIP:DIP-8_W7.62mm
Connections:
- net labels added: SPI_CLK, SPI_MOSI
- wire segments 49 -> 68
- no-connect marks 2 -> 6
Other:
- note added: "H1\nH3\nJ2\nJ1\nGND"
- note added: "H2\nJ3\nK1\nK4\nGND"

Commit message: update rc network values after tuning
Parts:
- C8: value C -> 10n
- R5, R6: value R -> 1k
Changed lines of the file:
@@
 P 7900 4150
 F 0 "R5" V 7693 4150 50  0000 C CNN
-F 1 "R" V 7784 4150 50  0000 C CNN
+F 1 "1k" V 7784 4150 50  0000 C CNN
 F 2 "Resistor_SMD:R_0805_2012Metric_Pad1.20x1.40mm_HandSolder" V 7830 4150 50  0001 C CNN
 F 3 "~" H 7900 4150 50  0001 C CNN
@@
 P 8800 3700
 F 0 "R6" V 8593 3700 50  0000 C CNN
-F 1 "R" V 8684 3700 50  0000 C CNN
+F 1 "1k" V 8684 3700 50  0000 C CNN
 F 2 "Resistor_SMD:R_0805_2012Metric_Pad1.20x1.40mm_HandSolder" V 8730 3700 50  0001 C CNN
 F 3 "~" H 8800 3700 50  0001 C CNN
@@
 P 8450 4300
 F 0 "C8" H 8335 4254 50  0000 R CNN
-F 1 "C" H 8335 4345 50  0000 R CNN
+F 1 "10n" H 8335 4345 50  0000 R CNN
 F 2 "Capacitor_SMD:C_0805_2012Metric_Pad1.18x1.45mm_HandSolder" H 8488 4150 50  0001 C CNN
 F 3 "~" H 8450 4300 50  0001 C CNN
